Commit message: Bumperbot py examples paketi oluşturuldu

File: bumperbot_description/urdf/bumperbot.urdf.xacro (robot description, xacro)
@@ -1,4 +1,5 @@
 <?xml version="1.0"?>
 <robot xmlns:xacro="http://www.ros.org/wiki/xacro" name="bumperbot">
+    <!--Vehicle Body Parameters -->
     <link name="base_footprint" />
     <link name="base_link">
@@ -7,5 +8,5 @@
             <geometry>
                 <!-- Hazır mesh kullanımı-->
-                <mesh filename="package://bumperbot_descripiton/meshes/base_link.STL"/>
+                <mesh filename="package://bumperbot_description/meshes/base_link.STL"/>
             </geometry>
         </visual>
@@ -16,3 +17,59 @@
         <origin xyz="0 0 0.033" rpy="0 0 0"/>
     </joint>
+    <link name="wheel_right_link">
+        <visual>
+            <origin xyz="0.0 0.0 0" rpy="${pi/2} 0 0"/>
+            <geometry>
+                <!-- Hazır mesh kullanımı-->
+                <mesh filename="package://bumperbot_description/meshes/wheel_right_link.STL"/>
+            </geometry>
+        </visual>
+    </link>
+    <joint name="wheel_right_joint" type="continuous">
+        <parent link="base_link"/>
+        <child link="wheel_right_link"/>
+        <origin xyz="0 -0.07 0" rpy="0 0 0"/>
+        <axis xyz="0 1 0"/>
+    </joint>
+    <link name="wheel_left_link">
+        <visual>
+            <origin xyz="0.0 0.0 0" rpy="-${pi/2} 0 0"/>
+            <geometry>
+                <!-- Hazır mesh kullanımı-->
+                <mesh filename="package://bumperbot_description/meshes/wheel_left_link.STL"/>
+            </geometry>
+        </visual>
+    </link>
+    <joint name="wheel_left_joint" type="continuous">
+        <parent link="base_link"/>
+        <child link="wheel_left_link"/>
+        <origin xyz="0 0.07 0" rpy="0 0 0"/>
+        <axis xyz="0 1 0"/>
+    </joint>
+    <link name="caster_front_link">
+        <visual>
+            <origin xyz="0 0 0" rpy="0 0 0"/>
+            <geometry>
+                <mesh filename="package://bumperbot_description/meshes/caster_front_link.STL"/>
+            </geometry>
+        </visual>
+    </link>
+    <joint name="caster_front_joint" type="fixed">
+        <parent link="base_link"/>
+        <child link="caster_front_link"/>
+        <origin xyz="0.04755 0 -0.0275" rpy="0 0 0"/>
+    </joint>
+    <link name="caster_rear_link">
+        <visual>
+            <origin xyz="0 0 0" rpy="0 0 0"/>
+            <geometry>
+                <mesh filename="package://bumperbot_description/meshes/caster_rear_link.STL"/>
+            </geometry>
+        </visual>
+    </link>
+     <joint name="caster_rear_joint" type="fixed">
+        <parent link="base_link"/>
+        <child link="caster_rear_link"/>
+        <origin xyz="-0.04755 0 -0.0275" rpy="0 0 0"/>
+    </joint>
 </robot>

Commit message: Gazebo simülasyon ortamına robot düzgün bir şekilde spawn oldu

File: bumperbot_description/urdf/bumperbot.urdf.xacro (robot description, xacro)
@@ -1,75 +1,158 @@
 <?xml version="1.0"?>
-<robot xmlns:xacro="http://www.ros.org/wiki/xacro" name="bumperbot">
-    <!--Vehicle Body Parameters -->
-    <link name="base_footprint" />
+<robot name="bumperbot" xmlns:xacro="http://ros.org/wiki/xacro">
+    <!-- Include Gazebo Parameters -->
+    <xacro:include filename="$(find bumperbot_description)/urdf/bumperbot_gazebo.xacro"/>
+    <link name="base_footprint"/>
     <link name="base_link">
+        <inertial>
+            <origin xyz="0 0 0.04" rpy="0.0 0.25 0.3" />
+            <mass value="8.2573504e-01"/>
+            <inertia ixx="2.2124416e-02" ixy="-1.2294101e-04" ixz="3.4938785e-04"
+                    iyy="2.1193702e-02" iyz="-5.0120904e-05"
+                    izz="2.0064271e-02" />
+        </inertial>
         <visual>
-            <origin xyz="0 0 0" rpy="0 0 0"/>
+            <origin xyz="0 0 0" rpy="0 0 0" />
             <geometry>
-                <!-- Hazır mesh kullanımı-->
-                <mesh filename="package://bumperbot_description/meshes/base_link.STL"/>
+                <mesh filename="package://bumperbot_description/meshes/base_link.STL" />
             </geometry>
+            <material name="black"/>
         </visual>
+        <collision>
+            <origin xyz="0 0 0" rpy="0 0 0" />
+            <geometry>
+                <mesh filename="package://bumperbot_description/meshes/base_link.STL" />
+            </geometry>
+        </collision>
     </link>
     <joint name="base_joint" type="fixed">
         <parent link="base_footprint"/>
-        <child link="base_link"/>
+        <child link="base_link" />
         <origin xyz="0 0 0.033" rpy="0 0 0"/>
     </joint>
     <link name="wheel_right_link">
+        <inertial>
+            <origin xyz="0 -0.014 0" rpy="0 0 0" />
+            <mass value="0.0530086090966721" />
+            <inertia ixx="1.88176298336665E-05" ixy="-4.8444933029987E-10" ixz="1.88163708851143E-08"
+                    iyy="3.11510738647764E-05" iyz="-6.93560663069607E-11"
+                    izz="1.8801969558182E-05" />
+        </inertial>
         <visual>
-            <origin xyz="0.0 0.0 0" rpy="${pi/2} 0 0"/>
+            <origin xyz="0 0 0" rpy="1.57 0 0" />
             <geometry>
-                <!-- Hazır mesh kullanımı-->
-                <mesh filename="package://bumperbot_description/meshes/wheel_right_link.STL"/>
+                <mesh filename="package://bumperbot_description/meshes/wheel_right_link.STL" />
             </geometry>
+            <material name="blue"/>
         </visual>
+        <collision>
+            <origin xyz="0 -0.015 0" rpy="1.57 0 0" />
+            <geometry>
+                <sphere radius="0.033"/>
+            </geometry>
+        </collision>
     </link>
     <joint name="wheel_right_joint" type="continuous">
-        <parent link="base_link"/>
-        <child link="wheel_right_link"/>
-        <origin xyz="0 -0.07 0" rpy="0 0 0"/>
-        <axis xyz="0 1 0"/>
+        <origin xyz="0 -0.0701101849418637 0" rpy="0 0 0" />
+        <parent link="base_link" />
+        <child link="wheel_right_link" />
+        <axis xyz="0 1 0" />
     </joint>
-    <link name="wheel_left_link">
+    <link
+        name="wheel_left_link">
+        <inertial>
+            <origin xyz="0 0.014 0" rpy="0 0 0" />
+            <mass value="0.0530086043217644" />
+            <inertia ixx="1.8792911368909E-05"  ixy="3.31256392204584E-10" ixz="-1.14082001662767E-08"
+                    iyy="3.11510738759073E-05" iyz="-3.60499245082192E-10"
+                    izz="1.88266886146847E-05" />
+        </inertial>
         <visual>
-            <origin xyz="0.0 0.0 0" rpy="-${pi/2} 0 0"/>
+            <origin xyz="0 0 0" rpy="-1.57 0 0" />
             <geometry>
-                <!-- Hazır mesh kullanımı-->
-                <mesh filename="package://bumperbot_description/meshes/wheel_left_link.STL"/>
+                <mesh filename="package://bumperbot_description/meshes/wheel_left_link.STL" />
             </geometry>
+            <material name="blue"/>
         </visual>
+        <collision>
+            <origin xyz="0 0.015 0" rpy="-1.57 0 0" />
+            <geometry>
+                <sphere radius="0.033"/>
+            </geometry>
+        </collision>
     </link>
     <joint name="wheel_left_joint" type="continuous">
-        <parent link="base_link"/>
-        <child link="wheel_left_link"/>
-        <origin xyz="0 0.07 0" rpy="0 0 0"/>
-        <axis xyz="0 1 0"/>
+        <origin xyz="0 0.0701101849418642 0" rpy="0 0 0" />
+        <parent link="base_link" />
+        <child link="wheel_left_link" />
+        <axis xyz="0 1 0" />
     </joint>
     <link name="caster_front_link">
+        <inertial>
+        <origin xyz="3.89968128948481E-07 2.40073004698083E-07 0.00219173397061506" rpy="0 0 0" />
+        <mass value="1.44379265037903E-06" />
+        <inertia ixx="7.23075276010246E-11" ixy="-6.10956883467859E-16" ixz="2.22849693525031E-15"
+                iyy="3.8713793085917E-11"  iyz="2.93909858781952E-15"
+                izz="1.00967486676306E-10" />
+        </inertial>
         <visual>
-            <origin xyz="0 0 0" rpy="0 0 0"/>
+            <origin xyz="0 0 0" rpy="0 0 0" />
             <geometry>
-                <mesh filename="package://bumperbot_description/meshes/caster_front_link.STL"/>
+                <mesh filename="package://bumperbot_description/meshes/caster_front_link.STL" />
             </geometry>
+            <material name="silver"/>
         </visual>
+        <collision>
+            <origin xyz="0 0 0" rpy="0 0 0" />
+            <geometry>
+                <sphere radius="0.005"/>
+            </geometry>
+        </collision>
     </link>
     <joint name="caster_front_joint" type="fixed">
-        <parent link="base_link"/>
-        <child link="caster_front_link"/>
-        <origin xyz="0.04755 0 -0.0275" rpy="0 0 0"/>
+        <origin xyz="0.04755 0 -0.0275" rpy="0 0 0" />
+        <parent link="base_link" />
+        <child link="caster_front_link" />
+        <axis xyz="0 0 0" />
     </joint>
     <link name="caster_rear_link">
+        <inertial>
+            <origin xyz="3.8996812895542E-07 2.40073004698083E-07 0.00219173397061509" rpy="0 0 0" />
+            <mass value="1.44379265037902E-06" />
+            <inertia ixx="7.23075276010246E-11" ixy="-6.10956872363424E-16" ixz="2.22849693527207E-15"
+                    iyy="3.87137930859167E-11" iyz="2.939098587861E-15"
+                    izz="1.00967486676306E-10" />
+            </inertial>
         <visual>
-            <origin xyz="0 0 0" rpy="0 0 0"/>
+            <origin xyz="0 0 0" rpy="0 0 0" />
             <geometry>
-                <mesh filename="package://bumperbot_description/meshes/caster_rear_link.STL"/>
+                <mesh filename="package://bumperbot_description/meshes/caster_rear_link.STL" />
             </geometry>
+            <material name="silver"/>
         </visual>
+        <collision>
+            <origin xyz="0 0 0" rpy="0 0 0" />
+            <geometry>
+                <sphere radius="0.005"/>
+            </geometry>
+        </collision>
     </link>
-     <joint name="caster_rear_joint" type="fixed">
-        <parent link="base_link"/>
-        <child link="caster_rear_link"/>
-        <origin xyz="-0.04755 0 -0.0275" rpy="0 0 0"/>
+    <joint name="caster_rear_joint" type="fixed">
+        <origin xyz="-0.04755 0 -0.0275" rpy="0 0 0" />
+        <parent link="base_link" />
+        <child link="caster_rear_link" />
+        <axis xyz="0 0 0" />
     </joint>
+    <material name="blue">
+        <color rgba="0 0 1 1"/>
+    </material>
+    <material name="black">
+        <color rgba="0 0 0 1"/>
+    </material>
+    <material name="silver">
+        <color rgba="0.79 0.82 0.93 1"/>
+    </material>
+    <material name="dark_grey">
+        <color rgba="0.3 0.3 0.3 1"/>
+    </material>
 </robot>

Commit message: Imu sensörü başarıyla entegre edildi

File: bumperbot_description/urdf/bumperbot.urdf.xacro (robot description, xacro)
@@ -147,4 +147,30 @@
         <axis xyz="0 0 0" />
     </joint>
+    <link name="imu_link">
+        <inertial>
+            <origin xyz="-0.00552433659106688 0.000168210391520346 0.000514000497342681" rpy="0 0 0" />
+            <mass value="0.000528415362211671" />
+            <inertia ixx="1.46176048428261E-08" ixy="1.40015117949421E-10" ixz="-1.99633872937403E-12"
+                    iyy="8.59662482954888E-09" iyz="7.52375112767959E-12"
+                    izz="2.30279421279312E-08" />
+        </inertial>
+        <visual>
+            <origin xyz="0 0 0" rpy="0 0 0"/>
+            <geometry>
+                <mesh filename="package://bumperbot_description/meshes/imu_link.STL" />
+            </geometry>
+        </visual>
+        <collision>
+            <origin xyz="0 0 0" rpy="0 0 0"/>
+            <geometry>
+                <mesh filename="package://bumperbot_description/meshes/imu_link.STL"/>
+            </geometry>
+        </collision>
+    </link>
+    <joint name="imu_joint" type="fixed">
+        <origin xyz="0 0 0.07" rpy="3.14 0 0"/>
+        <parent link="base_link"/>
+        <child link="imu_link"/>
+    </joint>
     <material name="blue">
         <color rgba="0 0 1 1"/>

File: bumperbot_description/urdf/bumperbot_gazebo.xacro (robot description, xacro)
@@ -41,7 +41,8 @@
         <!-- ROS 2 Humble -->
         <xacro:if value="$(arg is_ignition)">
-        <plugin filename="ign_ros2_control-system" name="ign_ros2_control::IgnitionROS2ControlPlugin">
-            <parameters>$(find bumperbot_controller)/config/bumperbot_controllers.yaml</parameters>
-        </plugin>
+            <plugin filename="ign_ros2_control-system" name="ign_ros2_control::IgnitionROS2ControlPlugin">
+                <parameters>$(find bumperbot_controller)/config/bumperbot_controllers.yaml</parameters>
+            </plugin>
+            <plugin filename="ignition-gazebo-imu-system" name="ignition::gazebo::systems::Imu"></plugin>
         </xacro:if>
         <!-- ROS 2 Iron or above -->
@@ -52,3 +53,53 @@
         </xacro:unless>
     </gazebo>
+    <gazebo reference="imu_link">
+        <sensor name="imu" type="imu">
+            <always_on>true</always_on>
+            <update_rate>100</update_rate>
+            <gz_frame_id>imu_link</gz_frame_id>
+            <topic>imu</topic>
+            <imu>
+                <angular_velocity>
+                    <x>
+                        <noise type="gaussian">
+                            <mean>0.0</mean>
+                            <stddev>2e-4</stddev> <!-- variance -->
+                        </noise>
+                    </x>
+                    <y>
+                        <noise type="gaussian">
+                            <mean>0.0</mean>
+                            <stddev>2e-4</stddev>
+                        </noise>
+                    </y>
+                    <z>
+                        <noise type="gaussian">
+                            <mean>0.0</mean>
+                            <stddev>2e-4</stddev>
+                        </noise>
+                    </z>
+                </angular_velocity>
+                <linear_acceleration>
+                    <x>
+                        <noise type="gaussian">
+                            <mean>0.0</mean>
+                            <stddev>1e-7</stddev> <!-- variance -->
+                        </noise>
+                    </x>
+                    <y>
+                        <noise type="gaussian">
+                            <mean>0.0</mean>
+                            <stddev>1e-7</stddev> <!-- variance -->
+                        </noise>
+                    </y>
+                    <z>
+                        <noise type="gaussian">
+                            <mean>0.0</mean>
+                            <stddev>1e-7</stddev> <!-- variance -->
+                        </noise>
+                    </z>
+                </linear_acceleration>
+            </imu>
+        </sensor>
+    </gazebo>
 </robot>

Commit message: Imu orientation değeri düzeltildi. Ayrıca kalman filter node'u eklendi ve tek boyutlu tahmin yapıldı

File: bumperbot_description/urdf/bumperbot.urdf.xacro (robot description, xacro)
@@ -169,5 +169,5 @@
     </link>
     <joint name="imu_joint" type="fixed">
-        <origin xyz="0 0 0.07" rpy="3.14 0 0"/>
+        <origin xyz="0 0 0.0698986241758014" rpy="0 0 0"/>
         <parent link="base_link"/>
         <child link="imu_link"/>
